File: Hardware/SparkFun_MegaShield.sch (EAGLE design)
At the start: 21 parts, among them U1 ARDUINO-MEGAPROTO_SHIELD

Commit message: Ready for first review
Parts:
- removed U1: ARDUINO-MEGAPROTO_SHIELD, TempLibrary:ARDUINO-MEGAPROTO_SHIELD
- added JP1: AVR_SPI_PRG_6PTH, SparkFun-Connectors:AVR_SPI_PRG_6PTH
- added JP13: (no value), SparkFun-Connectors:M02PTH
- added JP14, JP2: (no value), SparkFun-Connectors:M01PTH
- added JP15: (no value), SparkFun-Connectors:M191X19
- added JP16: (no value), MegaProtoShield:M20
- added S2: SWITCH-MOMENTARY-2PTH, SparkFun-Electromechanical:SWITCH-MOMENTARY-2PTH
- added SJ1: JUMPER-PAD-2-NC_BY_TRACE, SparkFun-Passives:JUMPER-PAD-2-NC_BY_TRACE
- added SJ2, SJ3: JUMPER-PAD-2-NOYES_SILK, SparkFun-Passives:JUMPER-PAD-2-NOYES_SILK
- added U2: ARDUINO-MEGA_R3_SHIELD", MegaProtoShield:ARDUINO-MEGA_R3_SHIELD"
- JP10: device SparkFun:M06LOCK -> SparkFun-Connectors:M08
- JP11, JP12: device SparkFun:M02LOCK -> SparkFun-Connectors:M02PTH
- JP3: device SparkFun:M08LOCK -> SparkFun-Connectors:M10SILK_FEMALE_PTH
- JP4, JP5, JP6, JP7: device SparkFun:M08LOCK -> SparkFun-Connectors:M08
- JP8, JP9: value M16LOCK -> (none); device SparkFun:M16LOCK -> SparkFun-Connectors:M16PTH
- LED1, LED2: device SparkFun:LED5MM -> SparkFun-LED:LED3MM
- S1: value (none) -> SWITCH-MOMENTARY-2PTH; device SparkFun:TAC_SWITCHPTH -> SparkFun-Electromechanical:SWITCH-MOMENTARY-2PTH
Connections:
- removed net 3.3: JP10.2
- removed net 5V@1: JP12.1, JP12.2
- removed net D14: JP5.8
- removed net D15: JP5.7
- removed net D16: JP5.6
- removed net D17: JP5.5
- removed net D18: JP5.4
- removed net D19: JP5.3
- removed net RES: JP10.1, R3.1, S1.3, S1.4
- new net 3.3V: JP10.4, SJ2.1, U2.3.3V
- new net MISO: JP1.1
- new net MOSI: JP1.4
- new net N$205: JP10.2, U2.IOREF
- new net N$245: JP13.2, R1.2
- new net N$250: JP14.1, R2.2
- new net RESET: JP1.5, JP10.3, S1.2, U2.RESET
- new net RX1: JP5.6, U2.19(RX1)
- new net RX2: JP5.4, U2.17(RX2)
- new net RX3: JP5.2, U2.15(RX3)
- new net SCK: JP1.3
- new net SW1: JP2.1, R3.1, S2.2
- new net TX0: JP4.2, U2.1(TX0)
- new net TX2: JP5.3, U2.16(TX2)
- new net TX3: JP5.1, U2.14(TX3)
- new net VCC: JP16.1, JP16.10, JP16.11, JP16.12, JP16.13, JP16.14, JP16.15, JP16.16, JP16.17, JP16.18, JP16.19, JP16.2, JP16.20, JP16.3, JP16.4, JP16.5, JP16.6, JP16.7, JP16.8, JP16.9, SJ1.2, SJ2.2, SJ3.2
- net 5V: now also JP1.2, JP10.5, JP12.1, JP12.2, SJ1.1, U2.5V@0, U2.5V@1, U2.5V@2; no longer JP10.3, R1.2
- net A0: now also U2.A0(RX0)
- net A1: now also U2.A1(TX0)
- net A10: now also U2.A10
- net A11: now also U2.A11
- net A12: now also U2.A12
- net A13: now also U2.A13
- net A14: now also U2.A14
- net A15: now also U2.A15
- net A2: now also U2.A2
- net A3: now also U2.A3
- net A4: now also U2.A4
- net A5: now also U2.A5
- net A6: now also U2.A6
- net A7: now also U2.A7
- net A8: now also U2.A8
- net A9: now also U2.A9
- net AREF: now also U2.AREF
- net D10: now also U2.10
- net D11: now also U2.11
- net D12: now also U2.12
- net D13: now also U2.13; no longer R2.2
- net D2: now also U2.2
- net D22: now also JP9.16, U2.22; no longer JP9.1
- net D23: now also U2.23
- net D24: now also JP9.15, U2.24; no longer JP9.2
- net D25: now also U2.25
- net D26: now also JP9.14, U2.26; no longer JP9.3
- net D27: now also U2.27
- net D28: now also JP9.13, U2.28; no longer JP9.4
- net D29: now also U2.29
- net D3: now also U2.3
- net D30: now also JP9.12, U2.30; no longer JP9.5
- net D31: now also U2.31
- net D32: now also JP9.11, U2.32; no longer JP9.6
- net D33: now also U2.33
- net D34: now also JP9.10, U2.34; no longer JP9.7
- net D35: now also U2.35
- net D36: now also JP9.9, U2.36; no longer JP9.8
- net D37: now also U2.37
- net D38: now also JP9.8, U2.38; no longer JP9.9
- net D39: now also U2.39
- net D4: now also U2.4
- net D40: now also JP9.7, U2.40; no longer JP9.10
- net D41: now also U2.41
- net D42: now also JP9.6, U2.42; no longer JP9.11
- net D43: now also U2.43
- net D44: now also JP9.5, U2.44; no longer JP9.12
- net D45: now also U2.45
- net D46: now also JP9.4, U2.46; no longer JP9.13
- net D47: now also U2.47
- net D48: now also JP9.3, U2.48; no longer JP9.14
- net D49: now also U2.49
- net D5: now also U2.5
- net D50: now also JP9.2, U2.50; no longer JP9.15
- net D51: now also U2.51
- net D52: now also JP9.1, U2.52; no longer JP9.16
- net D53: now also U2.53
- net D6: now also U2.6
- net D7: now also U2.7
- net D8: now also U2.8
- net D9: now also U2.9
- net GND: now also JP1.6, JP10.6, JP10.7, JP15.1, JP15.10, JP15.11, JP15.12, JP15.13, JP15.14, JP15.15, JP15.16, JP15.17, JP15.18, JP15.19, JP15.2, JP15.3, JP15.4, JP15.5, JP15.6, JP15.7, JP15.8, JP15.9, S2.1, U2.GND@0, U2.GND@1, U2.GND@2, U2.GND@3, U2.GND@4; no longer JP10.4, JP10.5, S1.2
- net RX0: now also U2.0(RX0)
- net SCL: now also JP3.10, JP5.8, U2.21(SCL), U2.SCL; no longer JP5.1
- net SDA: now also JP3.9, JP5.7, U2.20(SDA), U2.SDA; no longer JP5.2
- net TX1: now also JP5.5, U2.18(TX1); no longer JP4.2
- net VIN: now also JP10.8, SJ3.1, U2.VIN; no longer JP10.6
Other:
- moved on the sheet: JP11, JP12, JP4, JP5, JP6, JP7, JP8, JP9, R1, R2, R3
